Commit message: Add whole-body motion planning with mplib 0.2.1
- New 'whole_body' control mode: base position-controlled (not velocity)
- Planning URDFs: tidyverse_bare.urdf (whole-body), tidyverse_arm_planning.urdf (arm-only)
- Auto-generated SRDF files for collision pair filtering
- Sub-millimeter accuracy on both arm-only and whole-body planning
- Key: set_base_pose(robot.pose) to sync mplib/SAPIEN frames
- Action order: [arm(7), gripper(1), base(3)] for all joint modes
- Updated README with full motion planning docs and examples

File: tidyverse_arm_only.urdf (robot description, URDF)
Before this commit: robot tidyverse, 25 links, 24 joints
Links:
- removed link base_x_link
- removed link base_y_link
- removed link root
- link base_link: geometry collision box size=0.05 0.05 0.05
- link left_inner_finger: geometry collision box size=0.05 0.05 0.05
- link left_inner_finger_pad: geometry collision box size=0.022 0.00635 0.0375
- link left_inner_knuckle: geometry collision box size=0.05 0.05 0.05
- link left_outer_finger: geometry collision box size=0.05 0.05 0.05
- link left_outer_knuckle: geometry collision box size=0.05 0.05 0.05
- link panda_link0: geometry collision box size=0.05 0.05 0.05
- link panda_link1: geometry collision box size=0.05 0.05 0.05
- link panda_link2: geometry collision box size=0.05 0.05 0.05
- link panda_link3: geometry collision box size=0.05 0.05 0.05
- link panda_link4: geometry collision box size=0.05 0.05 0.05
- link panda_link5: geometry collision box size=0.05 0.05 0.05
- link panda_link6: geometry collision box size=0.05 0.05 0.05
- link panda_link7: geometry collision box size=0.05 0.05 0.05
- link right_inner_finger: geometry collision box size=0.05 0.05 0.05
- link right_inner_finger_pad: geometry collision box size=0.022 0.00635 0.0375
- link right_inner_knuckle: geometry collision box size=0.05 0.05 0.05
- link right_outer_finger: geometry collision box size=0.05 0.05 0.05
- link right_outer_knuckle: geometry collision box size=0.05 0.05 0.05
- link robotiq_arg2f_base_link: geometry collision box size=0.05 0.05 0.05
Joints:
- removed joint base_x_joint
- removed joint base_y_joint
- removed joint base_yaw_joint

File: tidyverse_arm_planning.urdf (robot description, URDF)
Before this commit: robot tidyverse, 25 links, 24 joints
Links:
- link base_link: geometry collision box size=0.05 0.05 0.05
- link left_inner_finger: geometry collision box size=0.05 0.05 0.05
- link left_inner_finger_pad: geometry collision box size=0.022 0.00635 0.0375
- link left_inner_knuckle: geometry collision box size=0.05 0.05 0.05
- link left_outer_finger: geometry collision box size=0.05 0.05 0.05
- link left_outer_knuckle: geometry collision box size=0.05 0.05 0.05
- link panda_link0: geometry collision box size=0.05 0.05 0.05
- link panda_link1: geometry collision box size=0.05 0.05 0.05
- link panda_link2: geometry collision box size=0.05 0.05 0.05
- link panda_link3: geometry collision box size=0.05 0.05 0.05
- link panda_link4: geometry collision box size=0.05 0.05 0.05
- link panda_link5: geometry collision box size=0.05 0.05 0.05
- link panda_link6: geometry collision box size=0.05 0.05 0.05
- link panda_link7: geometry collision box size=0.05 0.05 0.05
- link right_inner_finger: geometry collision box size=0.05 0.05 0.05
- link right_inner_finger_pad: geometry collision box size=0.022 0.00635 0.0375
- link right_inner_knuckle: geometry collision box size=0.05 0.05 0.05
- link right_outer_finger: geometry collision box size=0.05 0.05 0.05
- link right_outer_knuckle: geometry collision box size=0.05 0.05 0.05
- link robotiq_arg2f_base_link: geometry collision box size=0.05 0.05 0.05
Joints:
- joint base_x_joint: axis 1 0 0 -> (none); limit lower=-20 upper=20 effort=600 velocity=1.0 -> (none); type prismatic -> fixed
- joint base_y_joint: axis 0 1 0 -> (none); limit lower=-20 upper=20 effort=600 velocity=1.0 -> (none); type prismatic -> fixed
- joint base_yaw_joint: axis 0 0 1 -> (none); limit lower=-6.28318 upper=6.28318 effort=600 velocity=1.5 -> (none); type revolute -> fixed

File: tidyverse_bare.urdf (robot description, URDF)
Before this commit: robot tidyverse, 25 links, 24 joints
Links:
- link base_link: geometry collision box size=0.05 0.05 0.05
- link left_inner_finger: geometry collision box size=0.05 0.05 0.05
- link left_inner_finger_pad: geometry collision box size=0.022 0.00635 0.0375
- link left_inner_knuckle: geometry collision box size=0.05 0.05 0.05
- link left_outer_finger: geometry collision box size=0.05 0.05 0.05
- link left_outer_knuckle: geometry collision box size=0.05 0.05 0.05
- link panda_link0: geometry collision box size=0.05 0.05 0.05
- link panda_link1: geometry collision box size=0.05 0.05 0.05
- link panda_link2: geometry collision box size=0.05 0.05 0.05
- link panda_link3: geometry collision box size=0.05 0.05 0.05
- link panda_link4: geometry collision box size=0.05 0.05 0.05
- link panda_link5: geometry collision box size=0.05 0.05 0.05
- link panda_link6: geometry collision box size=0.05 0.05 0.05
- link panda_link7: geometry collision box size=0.05 0.05 0.05
- link right_inner_finger: geometry collision box size=0.05 0.05 0.05
- link right_inner_finger_pad: geometry collision box size=0.022 0.00635 0.0375
- link right_inner_knuckle: geometry collision box size=0.05 0.05 0.05
- link right_outer_finger: geometry collision box size=0.05 0.05 0.05
- link right_outer_knuckle: geometry collision box size=0.05 0.05 0.05
- link robotiq_arg2f_base_link: geometry collision box size=0.05 0.05 0.05

File: tidyverse_planning.urdf (robot description, URDF)
Before this commit: robot tidyverse, 25 links, 24 joints
Links:
- link left_inner_finger: geometry collision mesh filename=robotiq_meshes/collision/robotiq_arg2f_85_inner_finger.dae.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 scale=0.001 0.001 0.001; visual mesh filename=robotiq_meshes/visual/robotiq_arg2f_85_inner_finger.dae scale=0.001 0.001 0.001
- link left_inner_knuckle: geometry collision mesh filename=robotiq_meshes/collision/robotiq_arg2f_85_inner_knuckle.dae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 scale=0.001 0.001 0.001; visual mesh filename=robotiq_meshes/visual/robotiq_arg2f_85_inner_knuckle.dae scale=0.001 0.001 0.001
- link left_outer_finger: geometry collision mesh filename=robotiq_meshes/collision/robotiq_arg2f_85_outer_finger.dae.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 scale=0.001 0.001 0.001; visual mesh filename=robotiq_meshes/visual/robotiq_arg2f_85_outer_finger.dae scale=0.001 0.001 0.001
- link left_outer_knuckle: geometry collision mesh filename=robotiq_meshes/collision/robotiq_arg2f_85_outer_knuckle.dae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 scale=0.001 0.001 0.001; visual mesh filename=robotiq_meshes/visual/robotiq_arg2f_85_outer_knuckle.dae scale=0.001 0.001 0.001
- link right_inner_finger: geometry collision mesh filename=robotiq_meshes/collision/robotiq_arg2f_85_inner_finger.dae.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 scale=0.001 0.001 0.001; visual mesh filename=robotiq_meshes/visual/robotiq_arg2f_85_inner_finger.dae scale=0.001 0.001 0.001
- link right_inner_knuckle: geometry collision mesh filename=robotiq_meshes/collision/robotiq_arg2f_85_inner_knuckle.dae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 scale=0.001 0.001 0.001; visual mesh filename=robotiq_meshes/visual/robotiq_arg2f_85_inner_knuckle.dae scale=0.001 0.001 0.001
- link right_outer_finger: geometry collision mesh filename=robotiq_meshes/collision/robotiq_arg2f_85_outer_finger.dae.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 scale=0.001 0.001 0.001; visual mesh filename=robotiq_meshes/visual/robotiq_arg2f_85_outer_finger.dae scale=0.001 0.001 0.001
- link right_outer_knuckle: geometry collision mesh filename=robotiq_meshes/collision/robotiq_arg2f_85_outer_knuckle.dae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 scale=0.001 0.001 0.001; visual mesh filename=robotiq_meshes/visual/robotiq_arg2f_85_outer_knuckle.dae scale=0.001 0.001 0.001
