Commit message: Move base_link origin to directly below panda_link0 (on ground)
BREAKING: base_link XY now coincides with arm base XY.
- qpos[0:2] directly positions the arm base in XY (no lateral offset)
- Only Z offset (0.47225m) remains between base_link and panda_link0
- Simplifies teleport positioning: set qpos[0:2] = desired arm XY - root XY
- Updated all 3 URDFs: tidyverse.urdf, tidyverse_bare.urdf, tidyverse_arm_planning.urdf
- Deleted stale SRDF files (will auto-regenerate)
- Base visual/collision meshes shifted to compensate
- Old offset was (0.435, 0.254, 0.47225); new is (0, 0, 0.47225)

File: tidyverse.urdf (robot description, URDF)
Before this commit: robot tidyverse, 25 links, 24 joints
Joints:
- joint base_to_arm: origin xyz=0.435 0.254 0.47225 rpy=0 0 0 -> xyz=0 0 0.47225 rpy=0 0 0

File: tidyverse_arm_planning.urdf (robot description, URDF)
Before this commit: robot tidyverse, 25 links, 24 joints
Joints:
- joint base_to_arm: origin xyz=0.435 0.254 0.47225 rpy=0 0 0 -> xyz=0 0 0.47225 rpy=0 0 0

File: tidyverse_bare.urdf (robot description, URDF)
Before this commit: robot tidyverse, 25 links, 24 joints
Joints:
- joint base_to_arm: origin xyz=0.435 0.254 0.47225 rpy=0 0 0 -> xyz=0 0 0.47225 rpy=0 0 0
- joint base_x_joint: limit lower=-20 upper=20 effort=600 velocity=1.0 -> lower=-3 upper=3 effort=600 velocity=1.0
- joint base_y_joint: limit lower=-20 upper=20 effort=600 velocity=1.0 -> lower=-3 upper=3 effort=600 velocity=1.0
- joint base_yaw_joint: limit lower=-6.28318 upper=6.28318 effort=600 velocity=1.5 -> lower=-3.14159 upper=3.14159 effort=600 velocity=1.5
